File: HORNO_PCB/HORNO_PCB.kicad_sch (KiCad schematic)
At the start: 297 parts, among them J0_1 Terminales de tornillo espaci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, J0_10 Terminales de tornillo espaci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, J0_13 Terminales de tornillo espaci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, J0_14 Terminales de tornillo espaci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, J0_18 Terminales de tornillo espaci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, J0_2 Terminales de tornillo espaci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, J0_3 Terminales de tornillo espaci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, J0_5 Terminales de tornillo espaci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, J0_6 Terminales de tornillo espaci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, J0_9 Terminales de tornillo espaci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, J1 20 Pin 2.54mm Header Male Bre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, J10 Salida 1, J11 Salida 1, J12 Salida 2, J13 24 VDC, J2 20 Pin 2.54mm Header Male Bre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, J3 20 Pin 2.54mm Header Male Bre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, J4 20 Pin 2.54mm Header Male Bre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, J5 Salida 4, J6 5 VDC, J7 Salida 3, J8 24 VDC, J9 Salida 2, K1 Relay 1, K2 Relay 2, K6 Relay 4, K7 Relay 3, K8 Relay 2, K9 Relay 1, Q1 2N2222, Q2 2N2222, Q3 2N2222, Q4 2N2222, Q6 IRG4PF50W, Q7 IRG4PF50W, U1 TLP521-1, U10 LM741, U11 LM741, U12 LM741, U15 TLP250, U17 LM741, U18 LM741, U19 TLP250, U2 TLP521-1, U20 L298HN Multiwatt15 H, U25 UDN2981A, U3 TLP521-1, U4 TLP521-1, U5 TLP521-1, U6 TLP521-1, U7 TLP521-1, U8 TLP521-1, U9 LM741

Commit message: Hojas de datos y actualización del esquema
Parts:
- removed C12, C7: 100nF, Capacitor_THT:C_Disc_D5.1mm_W3.2mm_P5.00mm, symbol Device:C
- removed D15, D16, D17, D18, D19, D20, D21, D22: 1N4001, Diode_THT:D_DO-41_SOD81_P10.16mm_Horizontal, symbol Diode:1N4001
- removed J0_10, J0_9: Terminales de tornillo espaciados en 3.5mm, TerminalBlock_Phoenix:TerminalBlock_Phoenix_PT-1,5-3-3.5-H_1x03_P3.50mm_Horizontal, symbol Connector:Screw_Terminal_01x03
- removed J6: 5 VDC, TerminalBlock_Phoenix:TerminalBlock_Phoenix_MKDS-1,5-2-5.08_1x02_P5.08mm_Horizontal, symbol Connector:Screw_Terminal_01x02
- removed J8: 24 VDC, TerminalBlock_Phoenix:TerminalBlock_Phoenix_MKDS-1,5-2-5.08_1x02_P5.08mm_Horizontal, symbol Connector:Screw_Terminal_01x02
- removed PS1, PS4, PS6, PS7: MEE1S0515SC, Converter_DCDC:Converter_DCDC_Murata_MEE1SxxxxSC_THT, symbol Converter_DCDC:MEE1S0315SC
- removed PS2, PS3: MEE1S0505SC, Converter_DCDC:Converter_DCDC_Murata_MEE1SxxxxSC_THT, symbol Converter_DCDC:MEE1S0315SC
- removed PS8: MEE1S0303SC, Converter_DCDC:Converter_DCDC_Murata_MEE1SxxxxSC_THT, symbol Converter_DCDC:MEE1S0315SC
- removed PX111, PX112, PX113, PX58, PX60, PX61, PX64, PX65, PX68, PX70, PX71: ~, Connector_Wire:SolderWire-0.75sqmm_1x01_D1.25mm_OD2.3mm, symbol Connector:Screw_Terminal_01x01
- removed R39, R40: Depende de la aplicación puente H, Resistor_THT:R_Axial_DIN0309_L9.0mm_D3.2mm_P15.24mm_Horizontal, symbol Device:R_US
- removed U20: L298HN Multiwatt15 H, Package_TO_SOT_THT:TO-220-15_P2.54x2.54mm_StaggerOdd_Lead5.84mm_TabDown, symbol Driver_Motor:L298HN
- added PX85: ~, Connector_Wire:SolderWire-0.75sqmm_1x01_D1.25mm_OD2.3mm, symbol Connector:Screw_Terminal_01x01
Connections:
- net at C1.2, C2.2, C3.2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: now also J13.1 (Pin_1), PX45.1 (Pin_1), PX55.1 (Pin_1), PX74.1 (Pin_1), PX78.1 (Pin_1), PX79.1 (Pin_1), PX82.1 (Pin_1), U15.5 (VEE), U19.5 (VEE); no longer PX77.1 (Pin_1)
- net at PX84.1 (Pin_1): now also D10.2 (A), D11.2 (A), D12.2 (A), D13.2 (A), D14.2 (A), D9.2 (A), J13.2 (Pin_2), K1.5, K2.5, K6.5, K7.5, K8.5, K9.5, U25.9 (Vs), PX85.1 (Pin_1)
- net at J0_18.3 (Pin_3), Q6.3 (E): now also 3V3a1.1 (Pin_1), 5Va1.1 (Pin_1), C1.1, J0_14.3 (Pin_3), J1.2 (Pin_2), J1.3 (Pin_3), PX69.1 (Pin_1), PX75.1 (Pin_1), Q7.3 (E), R1.2, R2.2, R3.2, R4.2, R5.2, R6.2, R7.2, R8.2
- net at U10.4 (V-), U11.4 (V-), U12.4 (V-)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: now also PX77.1 (Pin_1)
- net at U10.7 (V+), U11.7 (V+), U12.7 (V+)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: now also PX83.1 (Pin_1), U15.8 (VCC), U19.8 (VCC)
- net at PX62.1 (Pin_1): now also Q1.3 (C), Q2.3 (C), Q3.3 (C), Q4.3 (C)
- now unconnected: PX76.1 (Pin_1)
Other:
- note added: "+12 voltios"
- note added: "-12 voltios"
- note added: "12 VDC"
- note removed: "+15 voltios"
- note removed: "-15 voltios"
- note removed: "5 voltios"
- moved on the sheet: C8, C9, J0_13, J0_14, J0_18, Q6, Q7, R19, R20, R21, R22, R23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

Commit message: Asignación de pines y actualización de esquematico
Parts:
- removed 3V3a1, 3V3b1, 5Va1, 5Vb1, P0, P12, P13, P14, P15, P16, P17, P18, P19, P2, P21, P22, P23, P25, P26, P27, P32, P33, P34, P35, P36, P37, P38, P39, P4, P5, PX1, PX10, PX11, PX118, PX119, PX12, PX121, PX122, PX123, PX124, PX13, PX14, PX15, PX16, PX17, PX18, PX19, PX2, PX20, PX21, PX22, PX23, PX24, PX25, PX26, PX27, PX28, PX29, PX3, PX30, PX31, PX32, PX33, PX34, PX35, PX36, PX37, PX38, PX39, PX4, PX40, PX41, PX42, PX43, PX44, PX46, PX47, PX48, PX49, PX5, PX50, PX51, PX52, PX53, PX54, PX56, PX57, PX59, PX6, PX63, PX66, PX67, PX7, PX72, PX8, PX80, PX9, RST1, RX1, TX1: ~, Connector_Wire:SolderWire-0.75sqmm_1x01_D1.25mm_OD2.3mm, symbol Connector:Screw_Terminal_01x01
- removed C1, C2: 100nF, Capacitor_THT:C_Disc_D5.1mm_W3.2mm_P5.00mm, symbol Device:C
- removed C3, C4: 10nF, Capacitor_THT:C_Disc_D5.1mm_W3.2mm_P5.00mm, symbol Device:C
- removed D5, D6, D7, D8: LED, LED_THT:LED_D4.0mm, symbol Device:LED
- removed J1, J2, J3, J4: 20 Pin 2.54mm Header Male Breakable, Connector_PinHeader_2.54mm:PinHeader_1x20_P2.54mm_Vertical, symbol Connector:Screw_Terminal_01x20
- removed J10, J11: Salida 1, TerminalBlock_Phoenix:TerminalBlock_Phoenix_MKDS-1,5-2-5.08_1x02_P5.08mm_Horizontal, symbol Connector:Screw_Terminal_01x02
- removed J12, J9: Salida 2, TerminalBlock_Phoenix:TerminalBlock_Phoenix_MKDS-1,5-2-5.08_1x02_P5.08mm_Horizontal, symbol Connector:Screw_Terminal_01x02
- removed J5: Salida 4, TerminalBlock_Phoenix:TerminalBlock_Phoenix_MKDS-1,5-2-5.08_1x02_P5.08mm_Horizontal, symbol Connector:Screw_Terminal_01x02
- removed J7: Salida 3, TerminalBlock_Phoenix:TerminalBlock_Phoenix_MKDS-1,5-2-5.08_1x02_P5.08mm_Horizontal, symbol Connector:Screw_Terminal_01x02
- removed Q3, Q4: 2N2222, Package_TO_SOT_THT:TO-92, symbol Transistor_BJT:2N2219
- removed R16, R17: 7.5KΩ - 1/4 W, Resistor_THT:R_Axial_DIN0207_L6.3mm_D2.5mm_P10.16mm_Horizontal, symbol Device:R_US
- removed R27, R32, R33, R34: 2.2 KΩ - 1/4 W, Resistor_THT:R_Axial_DIN0309_L9.0mm_D3.2mm_P15.24mm_Horizontal, symbol Device:R_US
- removed R35, R36: 39Ω - 1/4 W, Resistor_THT:R_Axial_DIN0207_L6.3mm_D2.5mm_P10.16mm_Horizontal, symbol Device:R_US
- removed R5, R6, R7, R8: 270Ω - 1/4 W, Resistor_THT:R_Axial_DIN0207_L6.3mm_D2.5mm_P10.16mm_Horizontal, symbol Device:R_US
- removed U11, U12: LM741, LM741_TH:LM741_TH, symbol Amplifier_Operational:LM741
- removed U5, U6, U7, U8: TLP521-1, Package_DIP:DIP-4_W7.62mm, symbol Isolator:Optocoupler_DC_PhotoNPN_AKEC
- added C10, C7: 100nF, Capacitor_THT:C_Disc_D5.1mm_W3.2mm_P5.00mm, symbol Device:C
- added CS1, CS2, CS3, IN1NEG, IN1POS, IN2NEG, IN2POS, IN3NEG, IN3POS, NC1, NC10, NC11, NC12, NC13, NC14, NC15, NC2, NC3, NC4, NC5, NC6, NC7, NC8, NC9, SCK1, SCK2, SCK3, SO1, SO2, SO3, VCC1, VCC2, VCC3: ~, Connector_Wire:SolderWire-0.75sqmm_1x01_D1.25mm_OD2.3mm, symbol Connector:Screw_Terminal_01x01
- added J0_10, J0_4, J0_7, J0_8, J0_9: Terminales de tornillo espaciados en 3.5mm, TerminalBlock_Phoenix:TerminalBlock_Phoenix_PT-1,5-3-3.5-H_1x03_P3.50mm_Horizontal, symbol Connector:Screw_Terminal_01x03
- renumbered 3V3a2 to 3V3a, 3V3b2 to 3V3b, 5Va2 to 5Va, 5Vb2 to 5Vb, P1 to P0, P31 to P12, P30 to P13, P40 to P14, P10 to P15, P28 to P16, P24 to P17, P8 to P18, P6 to P19, P11 to P2, P29 to P21, P3 to P22, P7 to P23, P43 to P25, P42 to P26, P41 to P27, P45 to P32, P44 to P33, P47 to P34, P46 to P35, P51 to P36, P50 to P37, P49 to P38, P48 to P39, P20 to P4, P9 to P5, RST2 to RST, RX2 to RX, TX2 to TX
Connections:
- net at J0_1.1 (Pin_1), U1.2, U2.2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: now also C5.2, C6.2, C8.2, C9.2, GND4.1 (Pin_1), GND6.1 (Pin_1), J0_13.2 (Pin_2), J0_3.3 (Pin_3), J0_5.3 (Pin_3), J13.1 (Pin_1), PX45.1 (Pin_1), PX55.1 (Pin_1), PX73.1 (Pin_1), PX74.1 (Pin_1), PX78.1 (Pin_1), PX79.1 (Pin_1), PX81.1 (Pin_1), PX82.1 (Pin_1), R21.2, R23.2, R37.2, R38.2, U1.3, U15.3 (C), U15.5 (VEE), U19.3 (C), U19.5 (VEE), U2.3, U25.10 (GND), U3.3, U4.3, C10.2, C7.2
- net at P5.1 (Pin_1): now also R11.2
- net at R26.2: now also P17.1 (Pin_1)
- net at J0_14.3 (Pin_3), J0_18.3 (Pin_3), PX69.1 (Pin_1)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: now also 5Va.1 (Pin_1), 5Vb.1 (Pin_1)
- net at R3.1, U3.4: now also P36.1 (Pin_1)
- net at K9.3: now also J0_7.2 (Pin_2)
- net at K9.1: now also J0_7.1 (Pin_1)
- net at Q2.1 (E), R37.1: now also P33.1 (Pin_1)
- net at C9.1, U18.3 (+): now also P26.1 (Pin_1)
- net at K1.3: now also J0_4.2 (Pin_2)
- net at K1.1: now also J0_4.1 (Pin_1)
- net at P32.1 (Pin_1): now also Q1.1 (E), R38.1
- net at C8.1, U17.3 (+): now also P25.1 (Pin_1)
- net at J0_6.1 (Pin_1): now also K2.1
- net at P12.1 (Pin_1): now also R44.2
- net at K1.4: now also J0_4.3 (Pin_3)
- net at P35.1 (Pin_1): now also R2.1, U2.4
- net at P16.1 (Pin_1): now also R20.2
- net at P39.1 (Pin_1): now also R4.1, U4.4
- net at J0_3.1 (Pin_1): now also RX.1 (Pin_1)
- net at PX62.1 (Pin_1), Q1.3 (C), Q2.3 (C): now also VCC1.1 (Pin_1), VCC2.1 (Pin_1), VCC3.1 (Pin_1)
- net at K8.3: now also J0_8.2 (Pin_2)
- net at K8.1: now also J0_8.1 (Pin_1)
- net at R46.2: now also P13.1 (Pin_1)
- net at K2.3: now also J0_6.2 (Pin_2)
- net at K2.4: now also J0_6.3 (Pin_3)
- net at P4.1 (Pin_1): now also R10.2
- net at P2.1 (Pin_1): now also R9.2
- net at GND5.1 (Pin_1): now also GND1.1 (Pin_1), GND2.1 (Pin_1), GND3.1 (Pin_1)
- net at 3V3b.1 (Pin_1): now also C10.1
- net at P23.1 (Pin_1): now also CS3.1 (Pin_1)
- net at P22.1 (Pin_1): now also CS2.1 (Pin_1)
- net at J0_3.2 (Pin_2): now also TX.1 (Pin_1)
- net at P34.1 (Pin_1): now also R1.1, U1.4
- net at K6.1: now also J0_10.1 (Pin_1)
- net at K6.3: now also J0_10.2 (Pin_2)
- net at K6.4: now also J0_10.3 (Pin_3)
- net at K9.4: now also J0_7.3 (Pin_3)
- net at R48.2: now also P14.1 (Pin_1)
- net at K7.1: now also J0_9.1 (Pin_1)
- net at K7.3: now also J0_9.2 (Pin_2)
- net at K7.4: now also J0_9.3 (Pin_3)
- net at K8.4: now also J0_8.3 (Pin_3)
- net at P21.1 (Pin_1): now also CS1.1 (Pin_1)
- net at 3V3a.1 (Pin_1): now also C7.1
- new net: SCK1.1 (Pin_1), SCK2.1 (Pin_1), SCK3.1 (Pin_1)
- new net: SO1.1 (Pin_1), SO2.1 (Pin_1), SO3.1 (Pin_1)
Other:
- note removed: "ESP32"
- note removed: "Otro ESP32 u otros modulos"
- moved on the sheet: J0_3

Commit message: Actualizacion de esquematico
Parts:
- removed J0_1, J0_2: Terminales de tornillo espaciados en 3.5mm, TerminalBlock_Phoenix:TerminalBlock_Phoenix_PT-1,5-3-3.5-H_1x03_P3.50mm_Horizontal, symbol Connector:Screw_Terminal_01x03
- removed J13: 24 VDC, TerminalBlock_Phoenix:TerminalBlock_Phoenix_MKDS-1,5-2-5.08_1x02_P5.08mm_Horizontal, symbol Connector:Screw_Terminal_01x02
- added J1, J2, J3, J4, J5, J6: switch, symbol Connector:Screw_Terminal_01x01
- added J7: 24VDC, symbol Connector:Screw_Terminal_01x03
- added R5, R6: 1 W, Resistor_THT:R_Axial_DIN0411_L9.9mm_D3.6mm_P15.24mm_Horizontal, symbol Device:R_US
- R28: value 2.2 KΩ - 1/4 W -> 2.4 KΩ - 1/2 W
- renumbered VCC1 to CS1, VCC2 to CS2, VCC3 to CS3, CS1 to GND1, CS2 to GND2, CS3 to GND3, NC6 to IN1NEG, NC4 to IN1POS, NC10 to IN2NEG, NC8 to IN2POS, NC14 to IN3NEG, NC12 to IN3POS, IN2POS to NC10, IN3NEG to NC12, IN3POS to NC14, IN1NEG to NC4, IN1POS to NC6, IN2NEG to NC8, GND1 to SCK1, GND2 to SCK2, GND3 to SCK3, SCK1 to VCC1, SCK2 to VCC2, SCK3 to VCC3
Connections:
- net at J0_18.1 (Pin_1), Q6.2 (C): now also R5.2
- net at J0_18.2 (Pin_2): now also R5.1
- net at C10.2, C5.2, C6.2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: now also J7.3 (Pin_3)
- net at D10.2 (A), D11.2 (A), D12.2 (A)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: now also R31.1, J2.1 (Pin_1), J4.1 (Pin_1), J6.1 (Pin_1), J7.1 (Pin_1)
- net at R28.1: now also J1.1 (Pin_1)
- net at R29.1: now also J3.1 (Pin_1)
- net at R30.1: now also J5.1 (Pin_1)
- net at J0_14.1 (Pin_1), Q7.2 (C): now also R6.2
- net at J0_14.2 (Pin_2): now also R6.1
Other:
- note added: "VERIFICAR SE SE NECESITA UN CONECTOR MAS PARA LA ALIMENTACION CONFIRMAR EL TIPO DE CONECTOR"
