File: HORNO_PCB/HORNO_PCB.kicad_pcb (KiCad board)
At the start: 2 copper layers, 40 parts, among them J0_3 Terminales de tornillo espaci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, J24 Screw_Terminal_01x20

Commit message: Organizacion de modulos en PCB
Parts:
- removed 3V3a1, 3V3b1, 5Va1, 5Vb1, GND4, GND5, GND6, P0, P12, P13, P14, P15, P16, P17, P18, P19, P2, P21, P22, P23, P25, P26, P27, P32, P33, P34, P35, P36, P37, P38, P39, P4, P5, RST1, RX1, TX1: ~, TerminalBlock_MetzConnect:TerminalBlock_MetzConnect_360271_1x01_Horizontal_ScrewM3.0_Boxed
- added C5: 10nF, Capacitor_THT:C_Disc_D5.1mm_W3.2mm_P5.00mm, F.Cu at (-74.6, 140.2)
- added C6: 10nF, Capacitor_THT:C_Disc_D5.1mm_W3.2mm_P5.00mm, F.Cu at (-74.6, 145.0)
- added C8: 10nF, Capacitor_THT:C_Disc_D5.1mm_W3.2mm_P5.00mm, F.Cu at (378.2, 182.1)
- added C9: 10nF, Capacitor_THT:C_Disc_D5.1mm_W3.2mm_P5.00mm, F.Cu at (378.2, 186.8)
- added D1: LED, LED_THT:LED_D4.0mm, F.Cu at (-57.9, 32.3)
- added D10: LED, LED_THT:LED_D4.0mm, F.Cu at (395.9, 33.6)
- added D11: LED, LED_THT:LED_D4.0mm, F.Cu at (402.4, 27.1)
- added D12: LED, LED_THT:LED_D4.0mm, F.Cu at (402.4, 33.6)
- added D13: LED, LED_THT:LED_D4.0mm, F.Cu at (408.9, 27.1)
- added D14: LED, LED_THT:LED_D4.0mm, F.Cu at (408.9, 33.6)
- added D2: LED, LED_THT:LED_D4.0mm, F.Cu at (-57.9, 38.8)
- added D3: LED, LED_THT:LED_D4.0mm, F.Cu at (-57.9, 45.2)
- added D4: LED, LED_THT:LED_D4.0mm, F.Cu at (-57.9, 51.7)
- added D9: LED, LED_THT:LED_D4.0mm, F.Cu at (395.9, 27.1)
- added F1: Fuse, Fuse:Fuseholder_Cylinder-5x20mm_Schurter_0031_8201_Horizontal_Open, F.Cu at (139.6, 311.4)
- added J0_1: Terminales de tornillo espaciados en 5mm, TerminalBlock_Phoenix:TerminalBlock_Phoenix_PT-1,5-3-5.0-H_1x03_P5.00mm_Horizontal, F.Cu at (152.2, -139.0)
- added J0_10: Terminales de tornillo espaciados en 5mm, TerminalBlock_Phoenix:TerminalBlock_Phoenix_PT-1,5-3-5.0-H_1x03_P5.00mm_Horizontal, F.Cu at (367.1, 45.0)
- added J0_13: Terminales de tornillo espaciados en 5mm, TerminalBlock_Phoenix:TerminalBlock_Phoenix_PT-1,5-3-5.0-H_1x03_P5.00mm_Horizontal, F.Cu at (358.0, 195.8)
- added J0_14: Terminales de tornillo espaciados en 5mm, TerminalBlock_Phoenix:TerminalBlock_Phoenix_PT-1,5-3-5.0-H_1x03_P5.00mm_Horizontal, F.Cu at (367.8, 106.0)
- added J0_18: Terminales de tornillo espaciados en 5mm, TerminalBlock_Phoenix:TerminalBlock_Phoenix_PT-1,5-3-5.0-H_1x03_P5.00mm_Horizontal, F.Cu at (367.8, 117.3)
- added J0_4: Terminales de tornillo espaciados en 5mm, TerminalBlock_Phoenix:TerminalBlock_Phoenix_PT-1,5-3-5.0-H_1x03_P5.00mm_Horizontal, F.Cu at (367.1, -11.6)
- added J0_5: Terminales de tornillo espaciados en 5mm, TerminalBlock_Phoenix:TerminalBlock_Phoenix_PT-1,5-3-5.0-H_1x03_P5.00mm_Horizontal, F.Cu at (-79.2, 131.6)
- added J0_6: Terminales de tornillo espaciados en 5mm, TerminalBlock_Phoenix:TerminalBlock_Phoenix_PT-1,5-3-5.0-H_1x03_P5.00mm_Horizontal, F.Cu at (367.1, -0.23)
- added J0_7: Terminales de tornillo espaciados en 5mm, TerminalBlock_Phoenix:TerminalBlock_Phoenix_PT-1,5-3-5.0-H_1x03_P5.00mm_Horizontal, F.Cu at (367.1, 11.1)
- added J0_8: Terminales de tornillo espaciados en 5mm, TerminalBlock_Phoenix:TerminalBlock_Phoenix_PT-1,5-3-5.0-H_1x03_P5.00mm_Horizontal, F.Cu at (367.1, 22.4)
- added J0_9: Terminales de tornillo espaciados en 5mm, TerminalBlock_Phoenix:TerminalBlock_Phoenix_PT-1,5-3-5.0-H_1x03_P5.00mm_Horizontal, F.Cu at (367.1, 33.7)
- added J1: switch, TerminalBlock_MetzConnect:TerminalBlock_MetzConnect_360271_1x01_Horizontal_ScrewM3.0_Boxed, F.Cu at (-76.2, 33.7)
- added J10: switch, TerminalBlock_MetzConnect:TerminalBlock_MetzConnect_360271_1x01_Horizontal_ScrewM3.0_Boxed, F.Cu at (142.8, 291.8)
- added J11: switch, TerminalBlock_MetzConnect:TerminalBlock_MetzConnect_360271_1x01_Horizontal_ScrewM3.0_Boxed, F.Cu at (142.8, 301.1)
- added J12: switch, TerminalBlock_MetzConnect:TerminalBlock_MetzConnect_360271_1x01_Horizontal_ScrewM3.0_Boxed, F.Cu at (153.9, 273.1)
- added J13: switch, TerminalBlock_MetzConnect:TerminalBlock_MetzConnect_360271_1x01_Horizontal_ScrewM3.0_Boxed, F.Cu at (153.9, 282.4)
- added J14: switch, TerminalBlock_MetzConnect:TerminalBlock_MetzConnect_360271_1x01_Horizontal_ScrewM3.0_Boxed, F.Cu at (153.9, 291.8)
- added J15: switch, TerminalBlock_MetzConnect:TerminalBlock_MetzConnect_360271_1x01_Horizontal_ScrewM3.0_Boxed, F.Cu at (153.9, 301.1)
- added J16: switch, TerminalBlock_MetzConnect:TerminalBlock_MetzConnect_360271_1x01_Horizontal_ScrewM3.0_Boxed, F.Cu at (164.9, 273.1)
- added J17: switch, TerminalBlock_MetzConnect:TerminalBlock_MetzConnect_360271_1x01_Horizontal_ScrewM3.0_Boxed, F.Cu at (164.9, 282.4)
- added J18: switch, TerminalBlock_MetzConnect:TerminalBlock_MetzConnect_360271_1x01_Horizontal_ScrewM3.0_Boxed, F.Cu at (164.9, 291.8)
- added J19: switch, TerminalBlock_MetzConnect:TerminalBlock_MetzConnect_360271_1x01_Horizontal_ScrewM3.0_Boxed, F.Cu at (164.9, 301.1)
- added J2: switch, TerminalBlock_MetzConnect:TerminalBlock_MetzConnect_360271_1x01_Horizontal_ScrewM3.0_Boxed, F.Cu at (-76.2, 43.1)
- added J20: switch, TerminalBlock_MetzConnect:TerminalBlock_MetzConnect_360271_1x01_Horizontal_ScrewM3.0_Boxed, F.Cu at (176.0, 273.1)
- added J21: switch, TerminalBlock_MetzConnect:TerminalBlock_MetzConnect_360271_1x01_Horizontal_ScrewM3.0_Boxed, F.Cu at (176.0, 282.4)
- added J22: switch, TerminalBlock_MetzConnect:TerminalBlock_MetzConnect_360271_1x01_Horizontal_ScrewM3.0_Boxed, F.Cu at (176.0, 291.8)
- added J23: switch, TerminalBlock_MetzConnect:TerminalBlock_MetzConnect_360271_1x01_Horizontal_ScrewM3.0_Boxed, F.Cu at (176.0, 301.1)
- added J25: Screw_Terminal_01x20, Connector_PinHeader_2.54mm:PinHeader_1x20_P2.54mm_Vertical, F.Cu at (146.4, -141.7)
- added J26: Screw_Terminal_01x20, Connector_PinHeader_2.54mm:PinHeader_1x20_P2.54mm_Vertical, F.Cu at (146.4, -54.6)
- added J27: Screw_Terminal_01x20, Connector_PinHeader_2.54mm:PinHeader_1x20_P2.54mm_Vertical, F.Cu at (151.0, -54.6)
- added J3: switch, TerminalBlock_MetzConnect:TerminalBlock_MetzConnect_360271_1x01_Horizontal_ScrewM3.0_Boxed, F.Cu at (-76.2, 52.4)
- added J4: switch, TerminalBlock_MetzConnect:TerminalBlock_MetzConnect_360271_1x01_Horizontal_ScrewM3.0_Boxed, F.Cu at (-76.2, 61.8)
- added J5: switch, TerminalBlock_MetzConnect:TerminalBlock_MetzConnect_360271_1x01_Horizontal_ScrewM3.0_Boxed, F.Cu at (-76.2, 71.1)
- added J6: switch, TerminalBlock_MetzConnect:TerminalBlock_MetzConnect_360271_1x01_Horizontal_ScrewM3.0_Boxed, F.Cu at (-76.2, 80.5)
- added J7: 24VDC, TerminalBlock_Phoenix:TerminalBlock_Phoenix_PT-1,5-3-5.0-H_1x03_P5.00mm_Horizontal, F.Cu at (167.9, 310.8)
- added J8: switch, TerminalBlock_MetzConnect:TerminalBlock_MetzConnect_360271_1x01_Horizontal_ScrewM3.0_Boxed, F.Cu at (142.8, 273.1)
- added J9: switch, TerminalBlock_MetzConnect:TerminalBlock_MetzConnect_360271_1x01_Horizontal_ScrewM3.0_Boxed, F.Cu at (142.8, 282.4)
- added K1: Relay 1, Relay_THT:Relay_SPDT_Fujitsu_FTR-LYCA005x_FormC_Vertical, F.Cu at (382.5, -14.4)
- added K2: Relay 2, Relay_THT:Relay_SPDT_Fujitsu_FTR-LYCA005x_FormC_Vertical, F.Cu at (382.5, -7.66)
- added K6: Relay 4, Relay_THT:Relay_SPDT_Fujitsu_FTR-LYCA005x_FormC_Vertical, F.Cu at (382.5, -0.92)
- added K7: Relay 3, Relay_THT:Relay_SPDT_Fujitsu_FTR-LYCA005x_FormC_Vertical, F.Cu at (382.5, 5.83)
- added K8: Relay 2, Relay_THT:Relay_SPDT_Fujitsu_FTR-LYCA005x_FormC_Vertical, F.Cu at (382.5, 12.6)
- added K9: Relay 1, Relay_THT:Relay_SPDT_Fujitsu_FTR-LYCA005x_FormC_Vertical, F.Cu at (382.5, 19.3)
- added Q1: 2N2222, Package_TO_SOT_THT:TO-92, F.Cu at (-80.7, 141.1)
- added Q2: 2N2222, Package_TO_SOT_THT:TO-92, F.Cu at (-80.7, 146.9)
- added Q6: IRG4PF50W, Package_TO_SOT_THT:TO-247-3_Vertical, F.Cu at (384.6, 126.1)
- added Q7: IRG4PF50W, Package_TO_SOT_THT:TO-247-3_Vertical, F.Cu at (384.6, 132.7)
- added R1: 270Ω - 1/4 W, Resistor_THT:R_Axial_DIN0207_L6.3mm_D2.5mm_P10.16mm_Horizontal, F.Cu at (-51.9, 31.1)
- added R10: 1 kΩ - 1/4 W, Resistor_THT:R_Axial_DIN0207_L6.3mm_D2.5mm_P10.16mm_Horizontal, F.Cu at (382.2, 30.0)
- added R11: 1 kΩ - 1/4 W, Resistor_THT:R_Axial_DIN0207_L6.3mm_D2.5mm_P10.16mm_Horizontal, F.Cu at (382.2, 34.0)
- added R12: 2.4 KΩ - 1/2 W, Resistor_THT:R_Axial_DIN0309_L9.0mm_D3.2mm_P15.24mm_Horizontal, F.Cu at (-69.1, 67.5)
- added R14: 7.5KΩ - 1/4 W, Resistor_THT:R_Axial_DIN0207_L6.3mm_D2.5mm_P10.16mm_Horizontal, F.Cu at (-64.1, 128.6)
- added R15: 7.5KΩ - 1/4 W, Resistor_THT:R_Axial_DIN0207_L6.3mm_D2.5mm_P10.16mm_Horizontal, F.Cu at (-64.1, 132.6)
- added R19: 10Ω - 1/4 W, Resistor_THT:R_Axial_DIN0207_L6.3mm_D2.5mm_P10.16mm_Horizontal, F.Cu at (365.9, 125.7)
- added R2: 270Ω - 1/4 W, Resistor_THT:R_Axial_DIN0207_L6.3mm_D2.5mm_P10.16mm_Horizontal, F.Cu at (-51.9, 35.1)
- added R20: 270Ω - 1/4 W, Resistor_THT:R_Axial_DIN0207_L6.3mm_D2.5mm_P10.16mm_Horizontal, F.Cu at (365.9, 129.7)
- added R21: Depende de la aplicación salida analógica, Resistor_THT:R_Axial_DIN0207_L6.3mm_D2.5mm_P10.16mm_Horizontal, F.Cu at (373.1, 192.8)
- added R22: Depende de la aplicación salida analógica, Resistor_THT:R_Axial_DIN0207_L6.3mm_D2.5mm_P10.16mm_Horizontal, F.Cu at (373.1, 196.9)
- added R23: Depende de la aplicación salida analógica, Resistor_THT:R_Axial_DIN0207_L6.3mm_D2.5mm_P10.16mm_Horizontal, F.Cu at (373.1, 200.9)
- added R24: Depende de la aplicación salida analógica, Resistor_THT:R_Axial_DIN0207_L6.3mm_D2.5mm_P10.16mm_Horizontal, F.Cu at (373.1, 205.0)
- added R25: 10Ω - 1/4 W, Resistor_THT:R_Axial_DIN0207_L6.3mm_D2.5mm_P10.16mm_Horizontal, F.Cu at (365.9, 133.8)
- added R26: 270Ω - 1/4 W, Resistor_THT:R_Axial_DIN0207_L6.3mm_D2.5mm_P10.16mm_Horizontal, F.Cu at (365.9, 137.8)
- added R28: 2.4 KΩ - 1/2 W, Resistor_THT:R_Axial_DIN0309_L9.0mm_D3.2mm_P15.24mm_Horizontal, F.Cu at (-69.1, 72.2)
- added R3: 270Ω - 1/4 W, Resistor_THT:R_Axial_DIN0207_L6.3mm_D2.5mm_P10.16mm_Horizontal, F.Cu at (-51.9, 39.2)
- added R37: 39Ω - 1/4 W, Resistor_THT:R_Axial_DIN0207_L6.3mm_D2.5mm_P10.16mm_Horizontal, F.Cu at (-64.1, 136.7)
- added R38: 39Ω - 1/4 W, Resistor_THT:R_Axial_DIN0207_L6.3mm_D2.5mm_P10.16mm_Horizontal, F.Cu at (-64.1, 140.7)
- added R4: 270Ω - 1/4 W, Resistor_THT:R_Axial_DIN0207_L6.3mm_D2.5mm_P10.16mm_Horizontal, F.Cu at (-51.9, 43.2)
- added R44: 1 kΩ - 1/4 W, Resistor_THT:R_Axial_DIN0207_L6.3mm_D2.5mm_P10.16mm_Horizontal, F.Cu at (382.2, 38.1)
- added R46: 1 kΩ - 1/4 W, Resistor_THT:R_Axial_DIN0207_L6.3mm_D2.5mm_P10.16mm_Horizontal, F.Cu at (382.2, 42.1)
- added R48: 1 kΩ - 1/4 W, Resistor_THT:R_Axial_DIN0207_L6.3mm_D2.5mm_P10.16mm_Horizontal, F.Cu at (382.2, 46.2)
- added R5: 1 W, Resistor_THT:R_Axial_DIN0411_L9.9mm_D3.6mm_P15.24mm_Horizontal, F.Cu at (383.3, 115.3)
- added R6: 1 W, Resistor_THT:R_Axial_DIN0411_L9.9mm_D3.6mm_P15.24mm_Horizontal, F.Cu at (383.3, 120.4)
- added R7: 2.4 KΩ - 1/2 W, Resistor_THT:R_Axial_DIN0309_L9.0mm_D3.2mm_P15.24mm_Horizontal, F.Cu at (-69.1, 58.0)
- added R8: 2.4 KΩ - 1/2 W, Resistor_THT:R_Axial_DIN0309_L9.0mm_D3.2mm_P15.24mm_Horizontal, F.Cu at (-69.1, 62.8)
- added R9: 1 kΩ - 1/4 W, Resistor_THT:R_Axial_DIN0207_L6.3mm_D2.5mm_P10.16mm_Horizontal, F.Cu at (382.2, 25.9)
- added U1: TLP521-1, Package_DIP:DIP-4_W7.62mm, F.Cu at (-69.1, 31.1)
- added U10: LM741, LM741_TH:LM741_TH, F.Cu at (-65.9, 121.0)
- added U15: TLP250, Package_DIP:DIP-8_W7.62mm, F.Cu at (382.9, 103.0)
- added U17: LM741, LM741_TH:LM741_TH, F.Cu at (360.2, 185.3)
- added U18: LM741, LM741_TH:LM741_TH, F.Cu at (371.3, 185.3)
- added U19: TLP250, Package_DIP:DIP-8_W7.62mm, F.Cu at (393.7, 103.0)
- added U2: TLP521-1, Package_DIP:DIP-4_W7.62mm, F.Cu at (-69.1, 37.8)
- added U25: UDN2981A, Package_DIP:DIP-18_W7.62mm_LongPads, F.Cu at (412.5, -14.5)
- added U3: TLP521-1, Package_DIP:DIP-4_W7.62mm, F.Cu at (-69.1, 44.4)
- added U4: TLP521-1, Package_DIP:DIP-4_W7.62mm, F.Cu at (-69.1, 51.0)
- added U9: LM741, LM741_TH:LM741_TH, F.Cu at (-77.0, 121.0)
- moved J0_3 85.7 mm to (152.2, -127.7)
- moved C10 67.3 mm to (150.3, -114.2)
- moved C7 67.3 mm to (150.3, -119.0)
- moved J24 38.7 mm to (141.8, -141.7)
Connections:
- C7 pad 1: Net-(3V3a1-Pin_1) -> Net-(J24-Pin_3)
- C7 pad 2: Net-(GND4-Pin_1) -> Net-(J0_3-Pin_3)
- J0_3 pad 3: Net-(GND4-Pin_1) -> Net-(J0_3-Pin_3)
- J24 pad 1: unconnected-(J24-Pin_1-Pad1) -> Net-(J0_3-Pin_3)
- J24 pad 10: unconnected-(J24-Pin_10-Pad10) -> Net-(J24-Pin_10)
- J24 pad 11: unconnected-(J24-Pin_11-Pad11) -> Net-(J24-Pin_11)
- J24 pad 12: unconnected-(J24-Pin_12-Pad12) -> Net-(J24-Pin_12)
- J24 pad 13: unconnected-(J24-Pin_13-Pad13) -> Net-(J24-Pin_13)
- J24 pad 15: unconnected-(J24-Pin_15-Pad15) -> Net-(J24-Pin_15)
- J24 pad 16: unconnected-(J24-Pin_16-Pad16) -> Net-(J24-Pin_16)
- J24 pad 17: unconnected-(J24-Pin_17-Pad17) -> Net-(J24-Pin_17)
- J24 pad 18: unconnected-(J24-Pin_18-Pad18) -> Net-(J24-Pin_18)
- J24 pad 2: unconnected-(J24-Pin_2-Pad2) -> Net-(J0_1-Pin_1)
- J24 pad 3: unconnected-(J24-Pin_3-Pad3) -> Net-(J24-Pin_3)
- J24 pad 4: unconnected-(J24-Pin_4-Pad4) -> Net-(J24-Pin_4)
- J24 pad 5: unconnected-(J24-Pin_5-Pad5) -> Net-(J0_3-Pin_1)
- J24 pad 6: unconnected-(J24-Pin_6-Pad6) -> Net-(J0_3-Pin_2)
- J24 pad 9: unconnected-(J24-Pin_9-Pad9) -> Net-(J24-Pin_9)

Commit message: Organizacion de modulos en PCB
Connections:
- K1 pad 11: (no net) -> Net-(J0_4-Pin_2)
- K1 pad 12: (no net) -> Net-(J0_4-Pin_1)
- K1 pad 14: (no net) -> Net-(J0_4-Pin_3)
- K1 pad A1: (no net) -> Net-(D14-K)
- K1 pad A2: (no net) -> Net-(D10-A)
- K2 pad 11: (no net) -> Net-(J0_6-Pin_2)
- K2 pad 12: (no net) -> Net-(J0_6-Pin_1)
- K2 pad 14: (no net) -> Net-(J0_6-Pin_3)
- K2 pad A1: (no net) -> Net-(D13-K)
- K2 pad A2: (no net) -> Net-(D10-A)
- K6 pad 11: (no net) -> Net-(J0_10-Pin_2)
- K6 pad 12: (no net) -> Net-(J0_10-Pin_1)
- K6 pad 14: (no net) -> Net-(J0_10-Pin_3)
- K6 pad A1: (no net) -> Net-(D9-K)
- K6 pad A2: (no net) -> Net-(D10-A)
- K7 pad 11: (no net) -> Net-(J0_9-Pin_2)
- K7 pad 12: (no net) -> Net-(J0_9-Pin_1)
- K7 pad 14: (no net) -> Net-(J0_9-Pin_3)
- K7 pad A1: (no net) -> Net-(D10-K)
- K7 pad A2: (no net) -> Net-(D10-A)
- K8 pad 11: (no net) -> Net-(J0_8-Pin_2)
- K8 pad 12: (no net) -> Net-(J0_8-Pin_1)
- K8 pad 14: (no net) -> Net-(J0_8-Pin_3)
- K8 pad A1: (no net) -> Net-(D11-K)
- K8 pad A2: (no net) -> Net-(D10-A)
- K9 pad 11: (no net) -> Net-(J0_7-Pin_2)
- K9 pad 12: (no net) -> Net-(J0_7-Pin_1)
- K9 pad 14: (no net) -> Net-(J0_7-Pin_3)
- K9 pad A1: (no net) -> Net-(D12-K)
- K9 pad A2: (no net) -> Net-(D10-A)
Changed lines of the file:
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@@
 			(layers "*.Cu" "*.Mask")
 			(remove_unused_layers no)
+			(net 100 "Net-(J0_6-Pin_2)")
+			(pintype "passive")
 		)
 		(pad "12" thru_hole circle
@@
 			(layers "*.Cu" "*.Mask")
 			(remove_unused_layers no)
+			(net 99 "Net-(J0_6-Pin_1)")
+			(pintype "passive")
 		)
 		(pad "14" thru_hole circle
@@
 			(layers "*.Cu" "*.Mask")
 			(remove_unused_layers no)
+			(net 98 "Net-(J0_6-Pin_3)")
+			(pintype "passive")
 		)
 		(pad "A1" thru_hole rect
@@
 			(layers "*.Cu" "*.Mask")
 			(remove_unused_layers no)
+			(net 38 "Net-(D13-K)")
+			(pintype "passive")
 		)
 		(pad "A2" thru_hole circle
@@
 			(layers "*.Cu" "*.Mask")
 			(remove_unused_layers no)
+			(net 16 "Net-(D10-A)")
+			(pintype "passive")
 		)
 		(embedded_fonts no)
@@
 			(layers "*.Cu" "*.Mask")
 			(remove_unused_layers no)
+			(net 105 "Net-(J0_8-Pin_2)")
+			(pintype "passive")
 		)
 		(pad "12" thru_hole circle
@@
 			(layers "*.Cu" "*.Mask")
 			(remove_unused_layers no)
+			(net 106 "Net-(J0_8-Pin_1)")
+			(pintype "passive")
 		)
 		(pad "14" thru_hole circle
@@
 			(layers "*.Cu" "*.Mask")
 			(remove_unused_layers no)
+			(net 104 "Net-(J0_8-Pin_3)")
+			(pintype "passive")
 		)
 		(pad "A1" thru_hole rect
@@
 			(layers "*.Cu" "*.Mask")
 			(remove_unused_layers no)
+			(net 25 "Net-(D11-K)")
+			(pintype "passive")
 		)
 		(pad "A2" thru_hole circle
@@
 			(layers "*.Cu" "*.Mask")
 			(remove_unused_layers no)
+			(net 16 "Net-(D10-A)")
+			(pintype "passive")
 		)
 		(embedded_fonts no)
@@
 			(layers "*.Cu" "*.Mask")
 			(remove_unused_layers no)
+			(net 112 "Net-(J0_10-Pin_2)")
+			(pintype "passive")
 		)
 		(pad "12" thru_hole circle
@@
 			(layers "*.Cu" "*.Mask")
 			(remove_unused_layers no)
+			(net 110 "Net-(J0_10-Pin_1)")
+			(pintype "passive")
 		)
 		(pad "14" thru_hole circle
@@
 			(layers "*.Cu" "*.Mask")
 			(remove_unused_layers no)
+			(net 111 "Net-(J0_10-Pin_3)")
+			(pintype "passive")
 		)
 		(pad "A1" thru_hole rect
@@
 			(layers "*.Cu" "*.Mask")
 			(remove_unused_layers no)
+			(net 14 "Net-(D9-K)")
+			(pintype "passive")
 		)
 		(pad "A2" thru_hole circle
@@
 			(layers "*.Cu" "*.Mask")
 			(remove_unused_layers no)
+			(net 16 "Net-(D10-A)")
+			(pintype "passive")
 		)
 		(embedded_fonts no)
@@
 			(layers "*.Cu" "*.Mask")
 			(remove_unused_layers no)
+			(net 107 "Net-(J0_9-Pin_2)")
+			(pintype "passive")
 		)
 		(pad "12" thru_hole circle
@@
 			(layers "*.Cu" "*.Mask")
 			(remove_unused_layers no)
+			(net 108 "Net-(J0_9-Pin_1)")
+			(pintype "passive")
 		)
 		(pad "14" thru_hole circle
@@
 			(layers "*.Cu" "*.Mask")
 			(remove_unused_layers no)
+			(net 109 "Net-(J0_9-Pin_3)")
+			(pintype "passive")
 		)
 		(pad "A1" thru_hole rect
@@
 			(layers "*.Cu" "*.Mask")
 			(remove_unused_layers no)
+			(net 18 "Net-(D10-K)")
+			(pintype "passive")
 		)
 		(pad "A2" thru_hole circle
@@
 			(layers "*.Cu" "*.Mask")
 			(remove_unused_layers no)
+			(net 16 "Net-(D10-A)")
+			(pintype "passive")
 		)
 		(embedded_fonts no)
@@
 			(layers "*.Cu" "*.Mask")
 			(remove_unused_layers no)
+			(net 102 "Net-(J0_7-Pin_2)")
+			(pintype "passive")
 		)
 		(pad "12" thru_hole circle
@@
 			(layers "*.Cu" "*.Mask")
 			(remove_unused_layers no)
+			(net 101 "Net-(J0_7-Pin_1)")
+			(pintype "passive")
 		)
 		(pad "14" thru_hole circle
@@
 			(layers "*.Cu" "*.Mask")
 			(remove_unused_layers no)
+			(net 103 "Net-(J0_7-Pin_3)")
+			(pintype "passive")
 		)
 		(pad "A1" thru_hole rect
@@
 			(layers "*.Cu" "*.Mask")
 			(remove_unused_layers no)
+			(net 36 "Net-(D12-K)")
+			(pintype "passive")
 		)
 		(pad "A2" thru_hole circle
@@
 			(layers "*.Cu" "*.Mask")
 			(remove_unused_layers no)
+			(net 16 "Net-(D10-A)")
+			(pintype "passive")
 		)
 		(embedded_fonts no)
@@
 			(layers "*.Cu" "*.Mask")
 			(remove_unused_layers no)
+			(net 95 "Net-(J0_4-Pin_2)")
+			(pintype "passive")
 		)
 		(pad "12" thru_hole circle
@@
 			(layers "*.Cu" "*.Mask")
 			(remove_unused_layers no)
+			(net 96 "Net-(J0_4-Pin_1)")
+			(pintype "passive")
 		)
 		(pad "14" thru_hole circle
@@
 			(layers "*.Cu" "*.Mask")
 			(remove_unused_layers no)
+			(net 97 "Net-(J0_4-Pin_3)")
+			(pintype "passive")
 		)
 		(pad "A1" thru_hole rect
@@
 			(layers "*.Cu" "*.Mask")
 			(remove_unused_layers no)
+			(net 94 "Net-(D14-K)")
+			(pintype "passive")
 		)
 		(pad "A2" thru_hole circle
@@
 			(layers "*.Cu" "*.Mask")
 			(remove_unused_layers no)
+			(net 16 "Net-(D10-A)")
+			(pintype "passive")
 		)
 		(embedded_fonts no)

Commit message: Actualización de PCB
Parts:
- added J28: switch, TerminalBlock_MetzConnect:TerminalBlock_MetzConnect_360271_1x01_Horizontal_ScrewM3.0_Boxed, F.Cu at (306.4, 238.4)
- added J29: switch, TerminalBlock_MetzConnect:TerminalBlock_MetzConnect_360271_1x01_Horizontal_ScrewM3.0_Boxed, F.Cu at (280.2, 238.2)
- moved J25 473.5 mm to (418.1, 246.1), turned to 180 degrees
- moved R37 459.2 mm to (372.5, 279.2), turned to 180 degrees
- moved R38 456.1 mm to (372.6, 272.4), turned to 180 degrees
- moved R4 455.1 mm to (369.4, 215.4)
- moved Q2 454.2 mm to (354.2, 277.9), turned to -90 degrees
- moved R3 454.2 mm to (369.3, 209.1)
- moved Q1 453.8 mm to (354.1, 270.9), turned to -90 degrees
- moved R2 453.5 mm to (369.3, 203.2)
- moved R1 452.7 mm to (369.3, 197.0)
- moved D4 451.9 mm to (361.9, 219.0)
- moved D3 450.9 mm to (361.7, 210.3)
- moved D2 450.3 mm to (361.8, 201.9)
- moved D1 449.4 mm to (361.6, 193.4)
- moved U4 449.3 mm to (348.0, 218.1)
- moved U3 448.8 mm to (348.3, 209.4)
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Connections:
- R12 pad 1: Net-(D10-A) -> Net-(J28-Pin_1)
Other:
- board outline added: 407.9 x 406.6 mm

Commit message: Actualizacion de PCB
Parts:
- removed J1, J2, J28, J29, J3, J4, J5, J6: switch, TerminalBlock_MetzConnect:TerminalBlock_MetzConnect_360271_1x01_Horizontal_ScrewM3.0_Boxed
- added J0_11: Terminales de tornillo espaciados en 5mm, TerminalBlock_Phoenix:TerminalBlock_Phoenix_PT-1,5-3-5.0-H_1x03_P5.00mm_Horizontal, F.Cu at (278.9, 209.1)
- added J0_12: Terminales de tornillo espaciados en 5mm, TerminalBlock_Phoenix:TerminalBlock_Phoenix_PT-1,5-3-5.0-H_1x03_P5.00mm_Horizontal, F.Cu at (278.2, 237.7)
- added J0_15: Terminales de tornillo espaciados en 5mm, TerminalBlock_Phoenix:TerminalBlock_Phoenix_PT-1,5-3-5.0-H_1x03_P5.00mm_Horizontal, F.Cu at (278.0, 266.8)
- added J0_2: Terminales de tornillo espaciados en 5mm, TerminalBlock_Phoenix:TerminalBlock_Phoenix_PT-1,5-3-5.0-H_1x03_P5.00mm_Horizontal, F.Cu at (278.7, 180.7)
- moved J0_5 28.8 mm to (278.7, 296.7)
- moved R15 27.5 mm to (343.9, 306.8)
- moved C5 27.5 mm to (307.5, 306.1)
- moved C6 27.5 mm to (307.5, 291.4)
- moved Q1 27.5 mm to (352.9, 298.4)
- moved Q2 27.5 mm to (353.0, 305.4)
- moved R14 27.5 mm to (344.0, 299.7)
- moved R37 27.5 mm to (371.3, 306.7)
- moved R38 27.5 mm to (371.4, 299.9)
- moved U10 27.5 mm to (319.2, 308.8)
- moved U9 27.5 mm to (319.2, 294.2)
- moved J0_3 4.02 mm to (278.7, 150.1)

Commit message: Actualizacion de PCB
Parts:
- added J1: switch, TerminalBlock_MetzConnect:TerminalBlock_MetzConnect_360271_1x01_Horizontal_ScrewM3.0_Boxed, F.Cu at (312.6, 125.5)
Connections:
- J11 pad 1: Net-(J0_1-Pin_1) -> Net-(J11-Pin_1)
- J21 pad 1: Net-(J0_1-Pin_1) -> Net-(J11-Pin_1)
- J24 pad 2: Net-(J0_1-Pin_1) -> Net-(J11-Pin_1)
- J25 pad 19: Net-(J0_1-Pin_1) -> Net-(J11-Pin_1)
- R1 pad 2: Net-(J0_1-Pin_1) -> Net-(J11-Pin_1)
- R2 pad 2: Net-(J0_1-Pin_1) -> Net-(J11-Pin_1)
- R3 pad 2: Net-(J0_1-Pin_1) -> Net-(J11-Pin_1)
- R4 pad 2: Net-(J0_1-Pin_1) -> Net-(J11-Pin_1)
Changed lines of the file:
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@@
 	(net 158 "Net-(J0_15-Pin_1)")
 	(net 159 "unconnected-(J0_15-Pin_2-Pad2)")
+	(net 160 "Net-(J11-Pin_1)")
 	(footprint "LED_THT:LED_D4.0mm"
 		(layer "F.Cu")
@@
 			(layers "*.Cu" "*.Mask")
 			(remove_unused_layers no)
-			(net 5 "Net-(J0_1-Pin_1)")
+			(net 160 "Net-(J11-Pin_1)")
 			(pintype "passive")
 		)
@@
 			(layers "*.Cu" "*.Mask")
 			(remove_unused_layers no)
-			(net 5 "Net-(J0_1-Pin_1)")
+			(net 160 "Net-(J11-Pin_1)")
 			(pinfunction "Pin_1")
 			(pintype "passive")
@@
 			(layers "*.Cu" "*.Mask")
 			(remove_unused_layers no)
-			(net 5 "Net-(J0_1-Pin_1)")
+			(net 160 "Net-(J11-Pin_1)")
 			(pinfunction "Pin_1")
 			(pintype "passive")
@@
 			(layers "*.Cu" "*.Mask")
 			(remove_unused_layers no)
-			(net 5 "Net-(J0_1-Pin_1)")
+			(net 160 "Net-(J11-Pin_1)")
 			(pinfunction "Pin_19")
 			(pintype "passive")
@@
 		)
 	)
+	(footprint "TerminalBlock_MetzConnect:TerminalBlock_MetzConnect_360271_1x01_Horizontal_ScrewM3.0_Boxed"
+		(layer "F.Cu")
+		(at 312.6 125.5)
+		(descr "single screw terminal block Metz Connect 360271, block size 9x7.3mm, drill diameter 1.5mm, pad diameter 3mm, https://www.metz-connect.com/media/file/8a8a80ea6e17c2e6016e3b8ef7cd2d65.de.0/product_summary_u_contact_de_en_fr.pdf , script-generated using https://gitlab.com/kicad/libraries/kicad-footprint-generator/-/tree/master/scripts/TerminalBlock_MetzConnect")
+		(tags "THT single screw terminal block Metz Connect 360271 size 9x7.3mm drill 1.5mm pad 3mm")
+		(property "Reference" "J1"
+			(at 0 -4.77 0)
+			(layer "F.SilkS")
+			(effects
+				(font
+					(size 1 1)
+					(thickness 0.15)
+				)
+			)
+		)
+		(property "Value" "switch"
+			(at 0 4.77 0)
+			(layer "F.Fab")
+			(effects
+				(font
+					(size 1 1)
+					(thickness 0.15)
+				)
+			)
+		)
+		(property "Datasheet" "~"
+			(at 0 0 0)
+			(layer "F.Fab")
+			(hide yes)
+			(effects
+				(font
+					(size 1.27 1.27)
+					(thickness 0.15)
+				)
+			)
+		)
+		(property "Description" "Generic screw terminal, single row, 01x01, script generated (kicad-library-utils/schlib/autogen/connector/)"
+			(at 0 0 0)
+			(layer "F.Fab")
+			(hide yes)
+			(effects
+				(font
+					(size 1.27 1.27)
+					(thickness 0.15)
+				)
+			)
+		)
+		(property ki_fp_filters "TerminalBlock*:*")
+		(sheetname "/")
+		(sheetfile "HORNO_PCB.kicad_sch")
+		(attr through_hole)
+		(fp_line
+			(start -4.62 -3.77)
+			(end 4.62 -3.77)
+			(stroke
+				(width 0.12)
+				(type solid)
+			)
+			(layer "F.SilkS")
+		)
+		(fp_line
+			(start -4.62 3.77)
+			(end -4.62 -3.77)
+			(stroke
+				(width 0.12)
+				(type solid)
+			)
+			(layer "F.SilkS")
+		)
+		(fp_line
+			(start 4.62 -3.77)
+			(end 4.62 3.77)
+			(stroke
+				(width 0.12)
+				(type solid)
+			)
+			(layer "F.SilkS")
+		)
+		(fp_line
+			(start 4.62 3.77)
+			(end -4.62 3.77)
+			(stroke
+				(width 0.12)
+				(type solid)
+			)
+			(layer "F.SilkS")
+		)
+		(fp_rect
+			(start -5 -4.15)
+			(end 5 4.15)
+			(stroke
+				(width 0.05)
+				(type solid)
+			)
+			(fill no)
+			(layer "F.CrtYd")
+		)
+		(fp_line
+			(start -4.5 -3.65)
+			(end 4.5 -3.65)
+			(stroke
+				(width 0.1)
+				(type solid)
+			)
+			(layer "F.Fab")
+		)
+		(fp_line
+			(start -4.5 3.65)
+			(end -4.5 -3.65)
+			(stroke
+				(width 0.1)
+				(type solid)
+			)
+			(layer "F.Fab")
+		)
+		(fp_line
+			(start 1.273 -1.517)
+			(end -1.517 1.273)
+			(stroke
+				(width 0.1)
+				(type solid)
+			)
+			(layer "F.Fab")
+		)
+		(fp_line
+			(start 1.517 -1.273)
+			(end -1.273 1.517)
+			(stroke
+				(width 0.1)
+				(type solid)
+			)
+			(layer "F.Fab")
+		)
+		(fp_line
+			(start 4.5 -3.65)
+			(end 4.5 3.65)
+			(stroke
+				(width 0.1)
+				(type solid)
+			)
+			(layer "F.Fab")
+		)
+		(fp_line
+			(start 4.5 3.65)
+			(end -4.5 3.65)
+			(stroke
+				(width 0.1)
+				(type solid)
+			)
+			(layer "F.Fab")
+		)
+		(fp_circle
+			(center 0 0)
+			(end 2 0)
+			(stroke
+				(width 0.1)
+				(type solid)
+			)
+			(fill no)
+			(layer "F.Fab")
+		)
+		(fp_text user "${REFERENCE}"
+			(at 0 -4.77 0)
+			(layer "F.Fab")
+			(effects
+				(font
+					(size 1 1)
+					(thickness 0.15)
+				)
+			)
+		)
+		(pad "1" thru_hole circle
+			(at 0 0)
+			(size 3 3)
+			(drill 1.5)
+			(layers "*.Cu" "*.Mask")
+			(remove_unused_layers no)
+			(net 5 "Net-(J0_1-Pin_1)")
+			(pinfunction "Pin_1")
+			(pintype "passive")
+		)
+		(embedded_fonts no)
+		(model "${KICAD9_3DMODEL_DIR}/TerminalBlock_MetzConnect.3dshapes/TerminalBlock_MetzConnect_360271_1x01_Horizontal_ScrewM3.0_Boxed.step"
+			(offset
+				(xyz 0 0 0)
+			)
+			(scale
+				(xyz 1 1 1)
+			)
+			(rotate
+				(xyz 0 0 0)
+			)
+		)
+	)
 	(footprint "TerminalBlock_Phoenix:TerminalBlock_Phoenix_PT-1,5-3-5.0-H_1x03_P5.00mm_Horizontal"
 		(layer "F.Cu")
@@
 			(layers "*.Cu" "*.Mask")
 			(remove_unused_layers no)
-			(net 5 "Net-(J0_1-Pin_1)")
+			(net 160 "Net-(J11-Pin_1)")
 			(pinfunction "Pin_2")
 			(pintype "passive")
@@
 			(layers "*.Cu" "*.Mask")
 			(remove_unused_layers no)
-			(net 5 "Net-(J0_1-Pin_1)")
+			(net 160 "Net-(J11-Pin_1)")
 			(pintype "passive")
 		)
@@
 			(layers "*.Cu" "*.Mask")
 			(remove_unused_layers no)
-			(net 5 "Net-(J0_1-Pin_1)")
+			(net 160 "Net-(J11-Pin_1)")
 			(pintype "passive")
 		)
@@
 			(layers "*.Cu" "*.Mask")
 			(remove_unused_layers no)
-			(net 5 "Net-(J0_1-Pin_1)")
+			(net 160 "Net-(J11-Pin_1)")
 			(pintype "passive")
 		)

Commit message: Tamaño de PCB  y ruteo
Parts:
- J0_1: value Terminales de tornillo espaciados en 5mm -> Alimentacion dispositivo serial
- J1: value switch -> +5V +24V
- moved F1 178.5 mm to (363.5, 313.9), turned to 90 degrees
- moved J7 151.9 mm to (332.4, 307.3), turned to 90 degrees
- moved J0_1 112.5 mm to (375.7, 177.6), turned to 180 degrees
- moved R23 93.5 mm to (461.3, 367.1)
- moved J1 84.4 mm to (370.4, 187.0)
- moved J0_10 84.4 mm to (486.7, 182.1)
- moved J0_13 83.1 mm to (486.7, 356.9)
- moved C9 82.1 mm to (454.3, 370.9)
- moved J0_3 81.6 mm to (355.5, 177.6), turned to 180 degrees
- moved R21 79.3 mm to (461.3, 339.3)
- moved J16 77.8 mm to (311.9, 375.5)
- moved J17 77.8 mm to (332.9, 375.5)
- moved J8 77.8 mm to (332.9, 332.3)
- moved J9 77.8 mm to (311.9, 332.3)
- moved U18 76.2 mm to (465.1, 375.1)
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Routing:
- net Net-(J0_13-Pin_2): track 0.00 -> 877.8 mm, vias 0 -> 3
- net Net-(D10-A): track 0.00 -> 568.1 mm, vias 0 -> 1
- net Net-(J8-Pin_1): track 0.00 -> 360.1 mm, vias 0 -> 2
- net Net-(J11-Pin_1): track 0.00 -> 264.2 mm, vias 0 -> 1
- net Net-(J14-Pin_1): track 0.00 -> 247.8 mm, vias 0 -> 3
- net Net-(J25-Pin_8): track 0.00 -> 184.6 mm, vias 0 -> 1
- net Net-(J25-Pin_9): track 0.00 -> 160.4 mm, vias 0 -> 1
- net Net-(J13-Pin_1): track 0.00 -> 113.5 mm, vias 0 -> 1
- net Net-(J25-Pin_10): track 0.00 -> 112.3 mm, vias 0 -> 1
- net Net-(J24-Pin_18): track 0.00 -> 97.8 mm, vias 0 -> 1
- net Net-(J24-Pin_4): track 0.00 -> 96.8 mm
- net Net-(J24-Pin_17): track 0.00 -> 88.5 mm, vias 0 -> 1
- net Net-(J24-Pin_10): track 0.00 -> 80.2 mm
- net Net-(J25-Pin_11): track 0.00 -> 76.5 mm, vias 0 -> 1
- net Net-(D14-K): track 0.00 -> 75.9 mm
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Other:
- board size 407.9 x 406.6 mm -> 198 x 218 mm
