File: HORNO_PCB/HORNO_PCB.kicad_pcb (KiCad board)
At the start: 2 copper layers, 198 x 218 mm, 109 parts, among them J0_1 Alimentacion dispositivo seri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, J0_10 Terminales de tornillo espaci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, J0_11 Terminales de tornillo espaci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, J0_12 Terminales de tornillo espaci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, J0_13 Terminales de tornillo espaci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, J0_14 Terminales de tornillo espaci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, J0_15 Terminales de tornillo espaci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, J0_18 Terminales de tornillo espaci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, J0_2 Terminales de tornillo espaci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, J0_3 Terminales de tornillo espaci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, J0_4 Terminales de tornillo espaci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, J0_5 Terminales de tornillo espaci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, J0_6 Terminales de tornillo espaci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, J0_7 Terminales de tornillo espaci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, J0_8 Terminales de tornillo espaci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, J0_9 Terminales de tornillo espaci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, J1 +5V +24V, J10 switch, J11 switch, J12 switch, J13 switch, J14 switch, J15 switch, J16 switch, J17 switch, J18 switch, J19 switch, J20 switch, J21 switch, J22 switch, J23 switch, J24 Screw_Terminal_01x20, J25 Screw_Terminal_01x20, J26 Screw_Terminal_01x20, J27 Screw_Terminal_01x20, J7 24VDC, J8 switch, J9 switch, K1 Relay 1, K2 Relay 2, K6 Relay 4, K7 Relay 3, K8 Relay 2, K9 Relay 1, Q1 2N2222, Q2 2N2222, Q6 IRG4PF50W, Q7 IRG4PF50W, U1 TLP521-1, U10 LM741, U15 TLP250, U17 LM741, U18 LM741, U19 TLP250, U2 TLP521-1, U25 UDN2981A, U3 TLP521-1, U4 TLP521-1, U9 LM741

Commit message: PCB terminada (falta revision)
Routing:
- net Net-(J25-Pin_14): track 66.1 -> 55.6 mm
Other:
- board text added: "GND 5V 3.3V GND RX TX RST P0 P22 P19 P23 P18 P5 P15 P2 P4 P17 P16"
- board text added: "GND 5V 3.3V P36 P37 P38 P39 P34 P35 P32 P33 P25 P26 P27 P14 P12 P13 P21"
- board text added: "NC IN1POS NC IN1NEG NC NC NC IN2POS NC IN2NEG NC NC NC IN3POS NC IN3NEG NC NC NC NC"
- board text added: "SCK1 CS1 SO1 GND VCC NC SCK2 CS2 SO2 GND VCC NC SCK3 CS3 SO3 GND VCC NC NC NC"

Commit message: Diseño del PCB: finalizado
Routing:
- net Net-(J25-Pin_9): track 169.2 -> 164.9 mm
- net Net-(J24-Pin_11): track 85.2 -> 84.0 mm

Commit message: Archivos de fabricacion
Routing:
- net Net-(D10-A): track 594.1 -> 599.0 mm
- net Net-(J25-Pin_9): track 164.9 -> 160.5 mm
- net Net-(D13-K): track 43.6 -> 42.3 mm
- net Net-(J15-Pin_1): track 266.9 -> 268.0 mm
- net Net-(J0_13-Pin_2): track 851.1 -> 852.1 mm
Changed lines of the file:
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@@
 			(outputformat 1)
 			(mirror no)
-			(drillshape 1)
+			(drillshape 0)
 			(scaleselection 1)
-			(outputdirectory "")
+			(outputdirectory "Archivos_de_fabricacion/")
 		)
 	)
@@
 		(tags "LED")
 		(property "Reference" "D11"
-			(at 1.27 -3.46 0)
+			(at 5.74 -0.3 0)
 			(layer "F.SilkS")
 			(effects
@@
 		(tags "THT Terminal Block Phoenix PT-1,5-3-5.0-H pitch 5mm size 15x9mm drill 1.3mm pad 2.6mm")
 		(property "Reference" "J0_1"
-			(at 5 -5.12 0)
+			(at 4.6 6.3 0)
 			(layer "F.SilkS")
 			(effects
@@
 		(tags "LED")
 		(property "Reference" "D10"
-			(at 1.27 -3.46 0)
+			(at 5.84 -0.1 0)
 			(layer "F.SilkS")
 			(effects
@@
 		(tags "THT Terminal Block Phoenix PT-1,5-3-5.0-H pitch 5mm size 15x9mm drill 1.3mm pad 2.6mm")
 		(property "Reference" "J0_12"
-			(at 5 -5.12 90)
+			(at 7.2 -5.4 90)
 			(layer "F.SilkS")
 			(effects
@@
 		(tags "THT Terminal Block Phoenix PT-1,5-3-5.0-H pitch 5mm size 15x9mm drill 1.3mm pad 2.6mm")
 		(property "Reference" "J0_3"
-			(at 5 -5.12 0)
+			(at 5 6.4 0)
 			(layer "F.SilkS")
 			(effects
@@
 		(tags "THT single screw terminal block Metz Connect 360271 size 9x7.3mm drill 1.5mm pad 3mm")
 		(property "Reference" "J1"
-			(at 0 -4.77 0)
+			(at -6.2 0.2 0)
 			(layer "F.SilkS")
 			(effects
@@
 		(tags "THT Terminal Block Phoenix PT-1,5-3-5.0-H pitch 5mm size 15x9mm drill 1.3mm pad 2.6mm")
 		(property "Reference" "J0_15"
-			(at 5 -5.12 90)
+			(at 1.5 -5.12 90)
 			(layer "F.SilkS")
 			(effects
@@
 		(tags "LED")
 		(property "Reference" "D12"
-			(at 1.27 -3.46 0)
+			(at 5.94 -0.1 0)
 			(layer "F.SilkS")
 			(effects
@@
 		(tags "THT Terminal Block Phoenix PT-1,5-3-5.0-H pitch 5mm size 15x9mm drill 1.3mm pad 2.6mm")
 		(property "Reference" "J0_2"
-			(at 5 -5.12 90)
+			(at 7.4 -5.7 90)
 			(layer "F.SilkS")
 			(effects
@@
 		(tags "LED")
 		(property "Reference" "D13"
-			(at 1.27 -3.46 0)
+			(at 5.74 0.2 0)
 			(layer "F.SilkS")
 			(effects
@@
 		(tags "LED")
 		(property "Reference" "D9"
-			(at 1.27 -3.46 0)
+			(at 5.34 0.1 0)
 			(layer "F.SilkS")
 			(effects
@@
 		(tags "Resistor Axial_DIN0309 series Axial Horizontal pin pitch 15.24mm 0.5W = 1/2W length 9mm diameter 3.2mm")
 		(property "Reference" "R7"
-			(at 7.62 -1.85 0)
+			(at 7.62 -2.7 0)
 			(layer "F.SilkS")
 			(effects
@@
 		(tags "LED")
 		(property "Reference" "D14"
-			(at 1.27 -3.46 0)
+			(at 5.84 0.3 0)
 			(layer "F.SilkS")
 			(effects
@@
 		(tags "THT Terminal Block Phoenix PT-1,5-3-5.0-H pitch 5mm size 15x9mm drill 1.3mm pad 2.6mm")
 		(property "Reference" "J0_11"
-			(at 5 -5.12 90)
+			(at 4 -5.2 90)
 			(layer "F.SilkS")
 			(effects
@@
 	)
 	(segment
+		(start 342.3 277.8)
+		(end 338 273.5)
+		(width 1)
+		(layer "F.Cu")
+		(net 3)
+	)
+	(segment
 		(start 482.316 303.884)
 		(end 480.3 305.9)
@@
 	)
 	(segment
+		(start 352.273 277.8)
+		(end 342.3 277.8)
+		(width 1)
+		(layer "F.Cu")
+		(net 3)
+	)
+	(segment
 		(start 452.045 337.325)
 		(end 452.045 355.745)
@@
 	)
 	(segment
-		(start 353.482 276.591)
-		(end 341.091 276.591)
-		(width 1)
-		(layer "F.Cu")
-		(net 3)
-	)
-	(segment
 		(start 406.4 355.5)
 		(end 451.8 355.5)
@@
 	)
 	(segment
-		(start 341.091 276.591)
-		(end 338 273.5)
+		(start 353.482 276.591)
+		(end 352.273 277.8)
 		(width 1)
 		(layer "F.Cu")
@@
 	)
 	(segment
-		(start 321.6 197.7)
-		(end 326 202.1)
+		(start 320.4 230.1)
+		(end 326 235.7)
 		(width 1)
 		(layer "F.Cu")
@@
 	)
 	(segment
-		(start 321.4 206.7)
-		(end 321.4 214.3)
-		(width 1)
-		(layer "F.Cu")
-		(net 16)
-	)
-	(segment
 		(start 320.7 369.9)
 		(end 311.7 360.9)
@@
 	)
 	(segment
-		(start 321.6 189.7)
-		(end 321.6 197.7)
+		(start 320.6 196.7)
+		(end 326 202.1)
 		(width 1)
 		(layer "F.Cu")
@@
 	)
 	(segment
-		(start 321.8 231.5)
-		(end 326 235.7)
+		(start 326 185.3)
+		(end 320.6 190.7)
 		(width 1)
 		(layer "F.Cu")
@@
 	)
 	(segment
-		(start 326 235.7)
-		(end 309.481 252.219)
+		(start 323.6 202.1)
+		(end 319.5 206.2)
 		(width 1)
 		(layer "F.Cu")
@@
 	)
 	(segment
-		(start 449.4 208.38)
-		(end 450.22 209.2)
+		(start 326 235.7)
+		(end 309.481 252.219)
 		(width 1)
 		(layer "F.Cu")
@@
 	)
 	(segment
-		(start 326 185.3)
-		(end 321.6 189.7)
+		(start 449.4 208.38)
+		(end 450.22 209.2)
 		(width 1)
 		(layer "F.Cu")
@@
 	)
 	(segment
-		(start 326 218.9)
-		(end 321.8 223.1)
-		(width 1)
-		(layer "F.Cu")
-		(net 16)
-	)
-	(segment
 		(start 449.4 189.58)
 		(end 450.22 190.4)
@@
 	)
 	(segment
-		(start 321.4 214.3)
-		(end 326 218.9)
+		(start 319.5 206.2)
+		(end 319.5 212.4)
 		(width 1)
 		(layer "F.Cu")
@@
 	)
 	(segment
-		(start 326 202.1)
-		(end 321.4 206.7)
+		(start 449.4 254.5)
+		(end 449.4 264.78)
 		(width 1)
 		(layer "F.Cu")
@@
 	)
 	(segment
-		(start 449.4 254.5)
-		(end 449.4 264.78)
+		(start 319.5 212.4)
+		(end 326 218.9)
 		(width 1)
 		(layer "F.Cu")
@@
 	)
 	(segment
-		(start 449.4 254.5)
-		(end 450.22 253.68)
+		(start 326 218.9)
+		(end 320.4 224.5)
 		(width 1)
 		(layer "F.Cu")
@@
 	)
 	(segment
-		(start 321.8 223.1)
-		(end 321.8 231.5)
+		(start 449.4 254.5)
+		(end 450.22 253.68)
 		(width 1)
 		(layer "F.Cu")
@@
 	)
 	(segment
+		(start 320.4 224.5)
+		(end 320.4 230.1)
+		(width 1)
+		(layer "F.Cu")
+		(net 16)
+	)
+	(segment
+		(start 326 202.1)
+		(end 323.6 202.1)
+		(width 1)
+		(layer "F.Cu")
+		(net 16)
+	)
+	(segment
+		(start 320.6 190.7)
+		(end 320.6 196.7)
+		(width 1)
+		(layer "F.Cu")
+		(net 16)
+	)
+	(segment
 		(start 449.4 236.4)
 		(end 449.4 245.98)
@@
 	)
 	(segment
-		(start 436.021 228.172)
-		(end 436.021 226)
-		(width 0.2)
-		(layer "F.Cu")
-		(net 24)
-	)
-	(segment
 		(start 442.957 335.844)
 		(end 445.153 335.844)
@@
 		(net 24)
 	)
-	(segment
-		(start 436.021 226)
-		(end 436.021 228.172)
-		(width 0.2)
-		(layer "F.Cu")
-		(net 24)
-	)
 	(via
 		(at 445.153 335.844)
@@
 	(segment
 		(start 446.44 246.8)
-		(end 446.44 245.498)
-		(width 0.2)
-		(layer "F.Cu")
-		(net 38)
-	)
-	(segment
-		(start 446.44 246.8)
 		(end 444.738 246.8)
 		(width 1)
@@
 	)
 	(segment
-		(start 353.953 267.677)
-		(end 351.4 270.23)
+		(start 430.598 227.4)
+		(end 424.37 233.629)
 		(width 0.2)
 		(layer "F.Cu")
@@
 	)
 	(segment
-		(start 430.598 227.4)
-		(end 424.37 233.629)
+		(start 432.1 227.4)
+		(end 430.598 227.4)
 		(width 0.2)
 		(layer "F.Cu")
@@
 	)
 	(segment
-		(start 432.1 227.4)
-		(end 430.598 227.4)
+		(start 353.2 267.8)
+		(end 351.4 269.6)
 		(width 0.2)
 		(layer "F.Cu")
@@
 	)
 	(segment
+		(start 353.2 256.935)
+		(end 353.2 267.8)
+		(width 0.2)
+		(layer "F.Cu")
+		(net 51)
+	)
+	(segment
 		(start 424.37 233.629)
 		(end 424.37 275.998)
@@
 	)
 	(segment
+		(start 351.4 269.6)
+		(end 351.4 270.23)
+		(width 0.2)
+		(layer "F.Cu")
+		(net 51)
+	)
+	(segment
 		(start 470.84 339.86)
 		(end 468.7 337.72)
@@
 	(segment
 		(start 353.953 256.182)
-		(end 353.953 267.677)
+		(end 353.2 256.935)
 		(width 0.2)
 		(layer "F.Cu")
@@
 	)
 	(segment
+		(start 343.46 260.31)
+		(end 341.5 262.27)
+		(width 0.2)
+		(layer "F.Cu")
+		(net 86)
+	)
+	(segment
 		(start 422 329)
 		(end 437.65 313.35)
@@
 	)
 	(segment
-		(start 343.46 260.31)
-		(end 342.57 261.2)
+		(start 341.5 262.27)
+		(end 341.5 273.35)
 		(width 0.2)
 		(layer "F.Cu")
@@
 	)
 	(segment
-		(start 342.57 261.2)
-		(end 342.57 274.42)
-		(width 0.2)
-		(layer "F.Cu")
-		(net 86)
-	)
-	(segment
-		(start 342.57 274.42)
+		(start 341.5 273.35)
 		(end 343.46 275.31)
 		(width 0.2)
@@
 	)
 	(segment
+		(start 343.46 275.31)
+		(end 347.17 271.6)
+		(width 0.2)
+		(layer "B.Cu")
+		(net 86)
+	)
+	(segment
 		(start 461.521 346.319)
 		(end 461.521 371.361)
@@
 	)
 	(segment
-		(start 346.867 271.903)
-		(end 375.9 271.903)
+		(start 375.597 271.6)
+		(end 379.995 275.998)
 		(width 0.2)
 		(layer "B.Cu")
@@
 	)
 	(segment
-		(start 343.46 275.31)
-		(end 346.867 271.903)
-		(width 0.2)
-		(layer "B.Cu")
-		(net 86)
-	)
-	(segment
 		(start 383.186 312.251)
 		(end 383.652 311.785)
@@
 	)
 	(segment
-		(start 375.9 271.903)
-		(end 379.995 275.998)
+		(start 347.17 271.6)
+		(end 375.597 271.6)
 		(width 0.2)
 		(layer "B.Cu")

Commit message: Codigo de prueba (pendiente la correccion a la PCB
Parts:
- added R13: Depende de la aplicación salida analógica, Resistor_THT:R_Axial_DIN0207_L6.3mm_D2.5mm_P10.16mm_Horizontal, F.Cu at (527.4, 210.8)
- added R16: Depende de la aplicación salida analógica, Resistor_THT:R_Axial_DIN0207_L6.3mm_D2.5mm_P10.16mm_Horizontal, F.Cu at (527.4, 214.9)
- added R17: Depende de la aplicación salida analógica, Resistor_THT:R_Axial_DIN0207_L6.3mm_D2.5mm_P10.16mm_Horizontal, F.Cu at (527.4, 218.9)
- added R18: Depende de la aplicación salida analógica, Resistor_THT:R_Axial_DIN0207_L6.3mm_D2.5mm_P10.16mm_Horizontal, F.Cu at (527.4, 223.0)
- added R27: Depende de la aplicación salida analógica, Resistor_THT:R_Axial_DIN0207_L6.3mm_D2.5mm_P10.16mm_Horizontal, F.Cu at (527.4, 227.1)
- added R29: Depende de la aplicación salida analógica, Resistor_THT:R_Axial_DIN0207_L6.3mm_D2.5mm_P10.16mm_Horizontal, F.Cu at (527.4, 231.1)
Connections:
- C10 pad 2: Net-(J0_13-Pin_2) -> Net-(D10-K)
- C5 pad 2: Net-(J0_13-Pin_2) -> Net-(D10-K)
- C6 pad 2: Net-(J0_13-Pin_2) -> Net-(D10-K)
- C8 pad 2: Net-(J0_13-Pin_2) -> Net-(D10-K)
- C9 pad 2: Net-(J0_13-Pin_2) -> Net-(D10-K)
- D11 pad 1: Net-(D11-K) -> Net-(D10-K)
- D11 pad 2: Net-(D10-A) -> Net-(D11-A)
- D12 pad 1: Net-(D12-K) -> Net-(D10-K)
- D12 pad 2: Net-(D10-A) -> Net-(D12-A)
- D13 pad 1: Net-(D13-K) -> Net-(D10-K)
- D13 pad 2: Net-(D10-A) -> Net-(D13-A)
- D14 pad 1: Net-(D14-K) -> Net-(D10-K)
- D14 pad 2: Net-(D10-A) -> Net-(D14-A)
- D9 pad 1: Net-(D9-K) -> Net-(D10-K)
- D9 pad 2: Net-(D10-A) -> Net-(D9-A)
- F1 pad 1: Net-(D10-A) -> Net-(J0_11-Pin_3)
- J0_11 pad 3: Net-(D10-A) -> Net-(J0_11-Pin_3)
- J0_12 pad 3: Net-(D10-A) -> Net-(J0_11-Pin_3)
- J0_13 pad 2: Net-(J0_13-Pin_2) -> Net-(D10-K)
- J0_14 pad 3: Net-(J0_13-Pin_2) -> Net-(D10-K)
- J0_15 pad 3: Net-(D10-A) -> Net-(J0_11-Pin_3)
- J0_18 pad 3: Net-(J0_13-Pin_2) -> Net-(D10-K)
- J0_2 pad 3: Net-(D10-A) -> Net-(J0_11-Pin_3)
- J0_5 pad 3: Net-(J0_13-Pin_2) -> Net-(D10-K)
- J10 pad 1: Net-(J0_13-Pin_2) -> Net-(D10-K)
- J12 pad 1: Net-(J0_13-Pin_2) -> Net-(D10-K)
- J14 pad 1: Net-(J0_13-Pin_2) -> Net-(D10-K)
- J16 pad 1: Net-(J0_13-Pin_2) -> Net-(D10-K)
- J17 pad 1: Net-(D10-A) -> Net-(J0_11-Pin_3)
- J18 pad 1: Net-(J0_13-Pin_2) -> Net-(D10-K)
- J19 pad 1: Net-(D10-A) -> Net-(J0_11-Pin_3)
- J20 pad 1: Net-(J0_13-Pin_2) -> Net-(D10-K)
- J21 pad 1: Net-(D10-A) -> Net-(J0_11-Pin_3)
- J25 pad 20: Net-(J0_13-Pin_2) -> Net-(D10-K)
- J7 pad 3: Net-(J0_13-Pin_2) -> Net-(D10-K)
- J9 pad 1: Net-(J0_13-Pin_2) -> Net-(D10-K)
- K1 pad A1: Net-(D14-K) -> Net-(U25-O6)
- K1 pad A2: Net-(D10-A) -> Net-(D10-K)
- K2 pad A1: Net-(D13-K) -> Net-(U25-O5)
- K2 pad A2: Net-(D10-A) -> Net-(D10-K)
- K6 pad A1: Net-(D9-K) -> Net-(U25-O1)
- K6 pad A2: Net-(D10-A) -> Net-(D10-K)
- K7 pad A1: Net-(D10-K) -> Net-(U25-O2)
- K7 pad A2: Net-(D10-A) -> Net-(D10-K)
- K8 pad A1: Net-(D11-K) -> Net-(U25-O3)
- K8 pad A2: Net-(D10-A) -> Net-(D10-K)
- K9 pad A1: Net-(D12-K) -> Net-(U25-O4)
- K9 pad A2: Net-(D10-A) -> Net-(D10-K)
- Q6 pad 3: Net-(J0_13-Pin_2) -> Net-(D10-K)
- Q7 pad 3: Net-(J0_13-Pin_2) -> Net-(D10-K)
- R21 pad 2: Net-(J0_13-Pin_2) -> Net-(D10-K)
- R23 pad 2: Net-(J0_13-Pin_2) -> Net-(D10-K)
- R37 pad 2: Net-(J0_13-Pin_2) -> Net-(D10-K)
- R38 pad 2: Net-(J0_13-Pin_2) -> Net-(D10-K)
- U1 pad 2: Net-(J0_13-Pin_2) -> Net-(D10-K)
- U1 pad 3: Net-(J0_13-Pin_2) -> Net-(D10-K)
- U15 pad 3: Net-(J0_13-Pin_2) -> Net-(D10-K)
- U19 pad 3: Net-(J0_13-Pin_2) -> Net-(D10-K)
- U2 pad 2: Net-(J0_13-Pin_2) -> Net-(D10-K)
- U2 pad 3: Net-(J0_13-Pin_2) -> Net-(D10-K)
- U25 pad 10: Net-(J0_13-Pin_2) -> Net-(D10-K)
- U25 pad 13: Net-(D14-K) -> Net-(U25-O6)
- U25 pad 14: Net-(D13-K) -> Net-(U25-O5)
- U25 pad 15: Net-(D12-K) -> Net-(U25-O4)
- U25 pad 16: Net-(D11-K) -> Net-(U25-O3)
- U25 pad 17: Net-(D10-K) -> Net-(U25-O2)
- U25 pad 18: Net-(D9-K) -> Net-(U25-O1)
- U3 pad 2: Net-(J0_13-Pin_2) -> Net-(D10-K)
- U3 pad 3: Net-(J0_13-Pin_2) -> Net-(D10-K)
- U4 pad 2: Net-(J0_13-Pin_2) -> Net-(D10-K)
- U4 pad 3: Net-(J0_13-Pin_2) -> Net-(D10-K)
Routing:
- net Net-(D10-K): track 23.5 -> 1061.4 mm, vias 0 -> 1
- net Net-(J0_13-Pin_2): track 852.1 -> 0.00 mm, vias 1 -> 0
- net Net-(D14-K): track 60.5 -> 0.00 mm
- net Net-(D13-K): track 42.3 -> 0.00 mm
- net Net-(D9-K): track 40.7 -> 0.00 mm
- net Net-(D12-K): track 25.8 -> 0.00 mm
- net Net-(D11-K): track 16.5 -> 0.00 mm
